Commit message: plugin error fix

File: src/simubot_description/urdf/simubot_gazebo.xacro (robot description, xacro)
@@ -1,4 +1,5 @@
 <?xml version="1.0"?>
 <robot name="simubot" xmlns:xacro="http://ros.org/wiki/xacro">
+  <xacro:macro name="simubot_gazebo">
   <!-- Wheels -->
   <gazebo reference="wheel_left_link">
@@ -61,5 +62,4 @@
         <always_on>true</always_on>
         <update_rate>100</update_rate>
-        <gz_frame_id>imu_link</gz_frame_id>
         <topic>imu</topic>
         <imu>
@@ -107,3 +107,4 @@
     </sensor>
   </gazebo>
+  </xacro:macro>
 </robot>

File: src/simubot_description/urdf/simubot_ros2_control.xacro (robot description, xacro)
@@ -1,27 +1,28 @@
 <?xml version="1.0"?>
 <robot xmlns:xacro="http://www.ros.org/wiki/xacro" name="simubot">
-    <ros2_control name="RobotSystem" type="system">
-        <!-- ros2_control Gazebo -->
-        <xacro:if value="$(arg is_sim)">
-            <!-- ROS 2 Humble -->
-            <xacro:if value="$(arg is_ignition)">
+    <xacro:macro name="simubot_ros2_control">
+        <ros2_control name="RobotSystem" type="system">
+            <!-- ros2_control Gazebo -->
+            <xacro:if value="$(arg is_sim)">
+                <!-- ROS 2 Humble -->
+                <xacro:if value="$(arg is_ignition)">
+                    <hardware>
+                        <plugin>ign_ros2_control/IgnitionSystem</plugin>
+                    </hardware>
+                </xacro:if>
+                <!-- ROS 2 Iron or above -->
+                <xacro:unless value="$(arg is_ignition)">
+                    <hardware>
+                        <plugin>gz_ros2_control/GazeboSimSystem</plugin>
+                    </hardware>
+                </xacro:unless>
+            </xacro:if>
+            <!-- ros2_control Real Robot -->
+            <xacro:unless value="$(arg is_sim)">
                 <hardware>
-                    <plugin>ign_ros2_control/IgnitionSystem</plugin>
-                </hardware>
-            </xacro:if>
-            <!-- ROS 2 Iron or above -->
-            <xacro:unless value="$(arg is_ignition)">
-                <hardware>
-                    <plugin>gz_ros2_control/GazeboSimSystem</plugin>
+                    <plugin>simubot_firmware/SimubotInterface</plugin>
+                    <param name="port">/dev/ttyUSB0</param>
                 </hardware>
             </xacro:unless>
-        </xacro:if>
-        <!-- ros2_control Real Robot -->
-        <xacro:unless value="$(arg is_sim)">
-            <hardware>
-                <plugin>simubot_firmware/SimubotInterface</plugin>
-                <param name="port">/dev/ttyUSB0</param>
-            </hardware>
-        </xacro:unless>
         <!-- ros2_control Common Interfaces -->
         <joint name="wheel_right_joint">
@@ -41,4 +42,18 @@
             <state_interface name="velocity" />
         </joint>
+        <!-- IMU Sensor -->
+        <sensor name="imu">
+            <state_interface name="orientation.x"/>
+            <state_interface name="orientation.y"/>
+            <state_interface name="orientation.z"/>
+            <state_interface name="orientation.w"/>
+            <state_interface name="angular_velocity.x"/>
+            <state_interface name="angular_velocity.y"/>
+            <state_interface name="angular_velocity.z"/>
+            <state_interface name="linear_acceleration.x"/>
+            <state_interface name="linear_acceleration.y"/>
+            <state_interface name="linear_acceleration.z"/>
+        </sensor>
     </ros2_control>
+    </xacro:macro>
 </robot>
